File: va4.kicad_pcb (KiCad board)
At the start: 2 copper layers, 95.8 x 73.1 mm, 19 parts, among them J1 LED, J2 MJ-4PP-9, SW1 RESET_SWITCH, SW2 SW_PUSH, SW3 SW_PUSH, SW4 SW_PUSH, SW5 SW_PUSH, U1 ProMicro

Commit message: Encoder support v0.4
Parts:
- removed G*** (x2): LOGO, my:logo-va_13.5mm
- removed Ref** (x5): Val**, kbd:HOLE
- added H1: MountingHole, kbd:HOLE, F.Cu at (45.4, 63.8)
- added H2: MountingHole, kbd:HOLE, F.Cu at (47.1, 83.3)
- added H3: MountingHole, kbd:HOLE, F.Cu at (86.5, 70.1)
- added H4: MountingHole, kbd:HOLE, F.Cu at (118.4, 97.6)
- added H5: MountingHole, kbd:HOLE, F.Cu at (128.8, 81.7)
- added R1: 5k, Resistors:0805, B.Cu at (104.0, 85.7)
- added R2: 5k, Resistors:0805, B.Cu at (106.4, 90.0)
- added SW6: Rotary_Encoder_Switch, AcheronHardware:ALPS_EC11E, F.Cu at (116.2, 84.8)
- SW5: footprint kbd:MX_ALPS_PG1350_noLed -> keyswitches:MX_reversible
- moved D4 2.02 mm to (121.2, 76.2)
Connections:
- U1 pad 12: Net-(U1-Pad12) -> encA
- U1 pad 13: Net-(U1-Pad13) -> encB
Routing:
- net encB: track 0.00 -> 64.1 mm, vias 0 -> 5
- net encA: track 0.00 -> 56.4 mm, vias 0 -> 5
- net VCC: track 68.9 -> 96.9 mm, vias 5 -> 7
- net GND: track 86.3 -> 110.2 mm, vias 6 -> 12
- net Net-(U1-Pad13): track 19.6 -> 0.00 mm
- net Net-(U1-Pad12): track 17.5 -> 0.00 mm
- net col3: track 80.6 -> 76.1 mm
- net col1: track 103.1 -> 99.5 mm
- net col0: track 133.1 -> 129.8 mm
- net Net-(D4-Pad2): track 20.4 -> 22.5 mm
- net row0: track 152.2 -> 150.4 mm, vias 4 -> 5
- net col2: track 87.5 -> 88.4 mm
Other:
- board text added: "va4 @toby_net v0.4"
- board text removed: "va4 @toby_net v0.3"
