File: va4.sch (KiCad schematic (older format))
At the start: 12 parts, among them J1 LED, J2 MJ-4PP-9, SW1 RESET_SWITCH, SW2 SW_PUSH, SW3 SW_PUSH, SW4 SW_PUSH, SW5 SW_PUSH, U1 ProMicro

Commit message: Encoder support v0.4
Parts:
- added H1, H2, H3, H4, H5: MountingHole, kbd:HOLE, symbol Mechanical:MountingHole
- added R1, R2: 5k, Resistors:0805, symbol Device:R
- added SW6: Rotary_Encoder_Switch, AcheronHardware:ALPS_EC11E, symbol Device:Rotary_Encoder_Switch
- SW5: footprint kbd:MX_ALPS_PG1350_noLed -> keyswitches:MX_reversible
Connections:
- net labels added: encA, encB
- wire segments 28 -> 42
- no-connect marks 13 -> 11
Other:
- moved on the sheet: D2, D3, D4, SW3, SW4
Changed lines of the file:
@@
 EESchema Schematic File Version 4
-LIBS:va4-cache
-EELAYER 26 0
+EELAYER 30 0
 EELAYER END
 $Descr A4 11693 8268
@@
 NoConn ~ 2025 3050
 NoConn ~ 2025 3150
-NoConn ~ 2025 3250
-NoConn ~ 3425 3250
 NoConn ~ 3425 3150
 NoConn ~ 3425 3050
@@
 L kbd:SW_PUSH SW3
 U 1 1 5C053C7A
-P 5900 2675
-F 0 "SW3" H 5900 2930 50  0000 C CNN
-F 1 "SW_PUSH" H 5900 2839 50  0000 C CNN
-F 2 "kbd:MX_ALPS_PG1350_noLed" H 5900 2675 50  0001 C CNN
-F 3 "" H 5900 2675 50  0000 C CNN
-	1    5900 2675
-	1    0    0    -1
-$EndComp
-Text GLabel 5600 2425 1    50   Input ~ 0
+P 5875 2675
+F 0 "SW3" H 5875 2930 50  0000 C CNN
+F 1 "SW_PUSH" H 5875 2839 50  0000 C CNN
+F 2 "kbd:MX_ALPS_PG1350_noLed" H 5875 2675 50  0001 C CNN
+F 3 "" H 5875 2675 50  0000 C CNN
+	1    5875 2675
+	1    0    0    -1
+$EndComp
+Text GLabel 5575 2425 1    50   Input ~ 0
 col1
 $Comp
 L Device:D D2
 U 1 1 5C053C81
-P 6200 2825
-F 0 "D2" V 6246 2746 50  0000 R CNN
-F 1 "D" V 6155 2746 50  0000 R CNN
-F 2 "kbd:D3_TH_SMD" H 6200 2825 50  0001 C CNN
-F 3 "~" H 6200 2825 50  0001 C CNN
-	1    6200 2825
+P 6175 2825
+F 0 "D2" V 6221 2746 50  0000 R CNN
+F 1 "D" V 6130 2746 50  0000 R CNN
+F 2 "kbd:D3_TH_SMD" H 6175 2825 50  0001 C CNN
+F 3 "~" H 6175 2825 50  0001 C CNN
+	1    6175 2825
 	0    -1   -1   0
 $EndComp
-Wire Wire Line
-	5600 2425 5600 2675
-Wire Wire Line
-	5300 2975 6200 2975
 Connection ~ 5300 2975
 $Comp
 L kbd:SW_PUSH SW4
 U 1 1 5C05442A
-P 6800 2675
-F 0 "SW4" H 6800 2930 50  0000 C CNN
-F 1 "SW_PUSH" H 6800 2839 50  0000 C CNN
-F 2 "kbd:MX_ALPS_PG1350_noLed" H 6800 2675 50  0001 C CNN
-F 3 "" H 6800 2675 50  0000 C CNN
-	1    6800 2675
-	1    0    0    -1
-$EndComp
-Text GLabel 6500 2425 1    50   Input ~ 0
+P 6775 2675
+F 0 "SW4" H 6775 2930 50  0000 C CNN
+F 1 "SW_PUSH" H 6775 2839 50  0000 C CNN
+F 2 "kbd:MX_ALPS_PG1350_noLed" H 6775 2675 50  0001 C CNN
+F 3 "" H 6775 2675 50  0000 C CNN
+	1    6775 2675
+	1    0    0    -1
+$EndComp
+Text GLabel 6475 2425 1    50   Input ~ 0
 col2
-$Comp
-L Device:D D3
-U 1 1 5C054431
-P 7100 2825
-F 0 "D3" V 7146 2746 50  0000 R CNN
-F 1 "D" V 7055 2746 50  0000 R CNN
-F 2 "kbd:D3_TH_SMD" H 7100 2825 50  0001 C CNN
-F 3 "~" H 7100 2825 50  0001 C CNN
-	1    7100 2825
-	0    -1   -1   0
-$EndComp
-Wire Wire Line
-	6500 2425 6500 2675
-Connection ~ 6200 2975
+Connection ~ 6175 2975
 $Comp
 L kbd:SW_PUSH SW5
@@
 F 0 "SW5" H 7675 2930 50  0000 C CNN
 F 1 "SW_PUSH" H 7675 2839 50  0000 C CNN
-F 2 "kbd:MX_ALPS_PG1350_noLed" H 7675 2675 50  0001 C CNN
+F 2 "keyswitches:MX_reversible" H 7675 2675 50  0001 C CNN
 F 3 "" H 7675 2675 50  0000 C CNN
 	1    7675 2675
@@
 L Device:D D4
 U 1 1 5C05486C
-P 7975 2825
-F 0 "D4" V 8021 2746 50  0000 R CNN
-F 1 "D" V 7930 2746 50  0000 R CNN
-F 2 "kbd:D3_TH_SMD" H 7975 2825 50  0001 C CNN
-F 3 "~" H 7975 2825 50  0001 C CNN
-	1    7975 2825
+P 8175 2825
+F 0 "D4" V 8221 2746 50  0000 R CNN
+F 1 "D" V 8130 2746 50  0000 R CNN
+F 2 "kbd:D3_TH_SMD" H 8175 2825 50  0001 C CNN
+F 3 "~" H 8175 2825 50  0001 C CNN
+	1    8175 2825
 	0    -1   -1   0
 $EndComp
 Wire Wire Line
 	7375 2425 7375 2675
-Connection ~ 7100 2975
-Wire Wire Line
-	7100 2975 7975 2975
-Wire Wire Line
-	7075 2975 7100 2975
-Wire Wire Line
-	6200 2975 7100 2975
+$Comp
+L Device:Rotary_Encoder_Switch SW6
+U 1 1 5D6F2CCE
+P 7700 3675
+F 0 "SW6" V 7746 3445 50  0000 R CNN
+F 1 "Rotary_Encoder_Switch" V 7655 3445 50  0000 R CNN
+F 2 "AcheronHardware:ALPS_EC11E" H 7550 3835 50  0001 C CNN
+F 3 "~" H 7700 3935 50  0001 C CNN
+	1    7700 3675
+	0    -1   -1   0
+$EndComp
+$Comp
+L Device:R R1
+U 1 1 5D6F4E9B
+P 7500 4300
+F 0 "R1" H 7650 4250 50  0000 R CNN
+F 1 "5k" H 7650 4350 50  0000 R CNN
+F 2 "Resistors:0805" V 7430 4300 50  0001 C CNN
+F 3 "~" H 7500 4300 50  0001 C CNN
+	1    7500 4300
+	-1   0    0    1
+$EndComp
+$Comp
+L Device:R R2
+U 1 1 5D6F5ECD
+P 7900 4300
+F 0 "R2" H 7970 4346 50  0000 L CNN
+F 1 "5k" H 7970 4255 50  0000 L CNN
+F 2 "Resistors:0805" V 7830 4300 50  0001 C CNN
+F 3 "~" H 7900 4300 50  0001 C CNN
+	1    7900 4300
+	1    0    0    -1
+$EndComp
+$Comp
+L power:GND #PWR01
+U 1 1 5D6F61D9
+P 7700 4100
+F 0 "#PWR01" H 7700 3850 50  0001 C CNN
+F 1 "GND" H 7705 3927 50  0000 C CNN
+F 2 "" H 7700 4100 50  0001 C CNN
+F 3 "" H 7700 4100 50  0001 C CNN
+	1    7700 4100
+	1    0    0    -1
+$EndComp
+Wire Wire Line
+	7700 3975 7700 4100
+Wire Wire Line
+	7975 2675 8175 2675
+Text GLabel 7975 3375 2    50   Input ~ 0
+row0
+Wire Wire Line
+	7800 3375 7975 3375
+Text GLabel 7600 3250 1    50   Input ~ 0
+col3
+Wire Wire Line
+	7600 3375 7600 3250
+Wire Wire Line
+	7600 3975 7600 4150
+Wire Wire Line
+	7600 4150 7500 4150
+Wire Wire Line
+	7800 3975 7800 4150
+Wire Wire Line
+	7800 4150 7900 4150
+Wire Wire Line
+	7500 4450 7500 4550
+Wire Wire Line
+	7900 4450 7900 4550
+Wire Wire Line
+	7500 4550 7700 4550
+Wire Wire Line
+	7700 4550 7700 4625
+Connection ~ 7700 4550
+Wire Wire Line
+	7700 4550 7900 4550
+$Comp
+L power:VCC #PWR02
+U 1 1 5D7008C5
+P 7700 4625
+F 0 "#PWR02" H 7700 4475 50  0001 C CNN
+F 1 "VCC" H 7717 4798 50  0000 C CNN
+F 2 "" H 7700 4625 50  0001 C CNN
+F 3 "" H 7700 4625 50  0001 C CNN
+	1    7700 4625
+	-1   0    0    1
+$EndComp
+Wire Wire Line
+	7500 4150 7250 4150
+Connection ~ 7500 4150
+Wire Wire Line
+	7900 4150 8125 4150
+Connection ~ 7900 4150
+Text GLabel 2025 3250 0    50   Input ~ 0
+encA
+Text GLabel 7250 4150 0    50   Input ~ 0
+encA
+Text GLabel 8125 4150 2    50   Input ~ 0
+encB
+Text GLabel 3425 3250 2    50   Input ~ 0
+encB
+Wire Wire Line
+	5300 2975 6175 2975
+Wire Wire Line
+	7075 2975 8175 2975
+Wire Wire Line
+	6175 2975 7075 2975
+Connection ~ 7075 2975
+$Comp
+L Device:D D3
+U 1 1 5C054431
+P 7075 2825
+F 0 "D3" V 7121 2746 50  0000 R CNN
+F 1 "D" V 7030 2746 50  0000 R CNN
+F 2 "kbd:D3_TH_SMD" H 7075 2825 50  0001 C CNN
+F 3 "~" H 7075 2825 50  0001 C CNN
+	1    7075 2825
+	0    -1   -1   0
+$EndComp
+Wire Wire Line
+	6475 2675 6475 2425
+Wire Wire Line
+	5575 2675 5575 2425
+$Comp
+L Mechanical:MountingHole H1
+U 1 1 5DF5704C
+P 4950 3250
+F 0 "H1" H 5050 3296 50  0000 L CNN
+F 1 "MountingHole" H 5050 3205 50  0000 L CNN
+F 2 "kbd:HOLE" H 4950 3250 50  0001 C CNN
+F 3 "~" H 4950 3250 50  0001 C CNN
+	1    4950 3250
+	1    0    0    -1
+$EndComp
+$Comp
+L Mechanical:MountingHole H2
+U 1 1 5DF586F1
+P 4950 3475
+F 0 "H2" H 5050 3521 50  0000 L CNN
+F 1 "MountingHole" H 5050 3430 50  0000 L CNN
+F 2 "kbd:HOLE" H 4950 3475 50  0001 C CNN
+F 3 "~" H 4950 3475 50  0001 C CNN
+	1    4950 3475
+	1    0    0    -1
+$EndComp
+$Comp
+L Mechanical:MountingHole H3
+U 1 1 5DF58AA4
+P 5750 3250
+F 0 "H3" H 5850 3296 50  0000 L CNN
+F 1 "MountingHole" H 5850 3205 50  0000 L CNN
+F 2 "kbd:HOLE" H 5750 3250 50  0001 C CNN
+F 3 "~" H 5750 3250 50  0001 C CNN
+	1    5750 3250
+	1    0    0    -1
+$EndComp
+$Comp
+L Mechanical:MountingHole H4
+U 1 1 5DF592E8
+P 5750 3475
+F 0 "H4" H 5850 3521 50  0000 L CNN
+F 1 "MountingHole" H 5850 3430 50  0000 L CNN
+F 2 "kbd:HOLE" H 5750 3475 50  0001 C CNN
+F 3 "~" H 5750 3475 50  0001 C CNN
+	1    5750 3475
+	1    0    0    -1
+$EndComp
+$Comp
+L Mechanical:MountingHole H5
+U 1 1 5DF595D3
+P 6500 3250
+F 0 "H5" H 6600 3296 50  0000 L CNN
+F 1 "MountingHole" H 6600 3205 50  0000 L CNN
+F 2 "kbd:HOLE" H 6500 3250 50  0001 C CNN
+F 3 "~" H 6500 3250 50  0001 C CNN
+	1    6500 3250
+	1    0    0    -1
+$EndComp
 $EndSCHEMATC
